File: cad/dlr_carrier.kicad_sch (KiCad schematic)
At the start: 60 parts, among them J1 PV_IN, J10 YL-83, J11 DEBUG_UART, J2 BQ24650, J3 BAT, J4 LMR33630ADDA, J5 CM4_J2, J6 U.FL, J7 SIM, J8 FLIR_LEPTON, J9 SI1145, U1 AP2112K-3.3, U2 LP5907MFX-3.8, U3 BG770A-NA, U4 TXS0108E, U5 DHT22, U6 ADS1115

Commit message: 🔌 feat: J8 FFC + commissioning USB-C + schematic generator fixes
Per ADR-013 (proposed in 2026-05-10-flir-mounting-design.md):

SKiDL netlist:
- J8 footprint changes from 14-pin THT 2.54mm header → Hirose FH12-14S-0.5SH
  FFC connector (sensors.py). Pin map preserves the GroupGets 14-pin Lepton
  breakout signal order so the daughterboard can reuse it.
- New build_commissioning_usbc() adds a sealed industrial USB-C receptacle
  on the carrier for live thermal preview during integrator aim of the
  Lepton daughterboard tilt. UFP/device mode (5.1k Rd on CC1/CC2), VBUS NC.
- Second USB pair on CM4 J5 (pins 36/37) routes the commissioning USB
  signals; the truly-unused pin list shrinks accordingly.

Schematic generator (cad/schematic/schematic.py) fixes for ERC:
- _real_pin_position() wrapper around kicad_sch_api.get_pin_position to fix
  its missing symbol-to-sheet y-inversion (root cause of most pin_not_connected
  errors — labels were landing 25-50 mm off from the actual pin positions).
- Per-net y-mod-4 residue for power symbols so distinct power rails can never
  share a y-coordinate, blocking KiCad's y-coincidence ERC false-merge cascade.
- Column-stagger in _place_block so adjacent same-type components (e.g. C10/C11
  decoupling caps) don't align their pin y's.
- Removed >30-pin orphan-NC skip (was a workaround for the y-inversion bug).
- Skip PWR_FLAG for nets with a Power-output driver (avoid two-power-outputs
  ERC error).
- Replaced the diagonal PWR_FLAG wire with an axis-aligned segment.

ERC: 139 → 3 violations, kicad-cli sch erc exits 0.

Co-Authored-By: Claude Opus 4.7 (1M context) <noreply@anthropic.com>
Parts:
- added J12: USBC_COMMISSIONING, Connector_USB:USB_C_Receptacle_GCT_USB4085, symbol Connector:USB_C_Receptacle_USB2.0_14P
- added R12, R13: 5.1k, Resistor_SMD:R_0402_1005Metric, symbol Device:R
- J7: footprint Connector_JAE:JAE_SIM_Card_SF72S006 -> Connector_Card:microSIM_JAE_SF53S006VCBR2000
- J8: value FLIR_LEPTON -> FLIR_LEPTON_FFC; footprint Connector_PinHeader_2.54mm:PinHeader_1x14_P2.54mm_Vertical -> Connector_FFC-FPC:Hirose_FH12-14S-0.5SH_1x14-1MP_P0.50mm_Horizontal
Connections:
- net +3V3: now also J11.1 (Pin_1), J11.4 (Pin_4), J5.25 (Pin_25), J5.39 (Pin_39), J5.5 (Pin_5), J5.7 (Pin_7), J9.1 (Pin_1), R7.2, R8.2, U1.2 (GND), U2.2 (GND), U4.11 (GND), U4.19 (VCCB), U6.4 (AIN0), U6.8 (VDD), J12.A1 (GND), J12.A12 (GND), J12.B1 (GND), J12.B12 (GND), J12.S1 (SHIELD), R12.2, R13.2; no longer C1.1, C10.1, C12.1, C13.1, C14.1, C15.1, C16.1, C17.1, C18.1, C19.1, C2.1, C2.2, C20.1, C21.1, C22.1, C23.1, C3.1, C4.1, C5.1, C6.1, C6.2, C7.1, C8.1, C9.1, D1.1 (K), D1.2 (A), J1.1 (Pin_1), J10.4 (Pin_4), J11.2 (Pin_2), J11.3 (Pin_3), J2.10 (Pin_10), J2.12 (Pin_12), J2.14 (Pin_14), J2.2 (Pin_2), J2.3 (Pin_3), J2.4 (Pin_4), J2.5 (Pin_5), J2.6 (Pin_6), J2.7 (Pin_7), J3.1 (Pin_1), J4.1 (Pin_1), J4.2 (Pin_2), J4.3 (Pin_3), J4.6 (Pin_6), J4.8 (Pin_8), J5.10 (Pin_10), J5.12 (Pin_12), J5.13 (Pin_13), J5.15 (Pin_15), J5.16 (Pin_16), J5.18 (Pin_18), J5.21 (Pin_21), J5.22 (Pin_22), J5.24 (Pin_24), J5.26 (Pin_26), J5.27 (Pin_27), J5.28 (Pin_28), J5.29 (Pin_29), J5.31 (Pin_31), J5.32 (Pin_32), J5.33 (Pin_33), J5.35 (Pin_35), J5.36 (Pin_36), J5.37 (Pin_37), J5.38 (Pin_38), J5.40 (Pin_40), J5.8 (Pin_8), J6.1 (In), J7.6 (VPP), J7.7 (I/O), J8.11 (Pin_11), J8.2 (Pin_2), J8.4 (Pin_4), J8.5 (Pin_5), J8.6 (Pin_6), J9.5 (Pin_5), L1.1, L1.2, L2.1, L2.2, R1.1, R1.2, R2.1, R2.2, R3.1, R4.1, R5.1, R5.2, R6.1, R7.1, R8.1, U1.1 (VIN), U1.3 (EN), U2.1 (IN), U2.3 (EN), U3.52 (VBAT_RF), U3.53 (VBAT_RF), U3.87 (GPIO20), U4.13 (B7), U4.14 (B6), U4.16 (B4), U4.17 (B3), U4.9 (A8), U6.2 (ALERT/RDY), U6.6 (AIN2)
- net CELL_NET_1V8: now also U3.21 (NET_STATUS), U4.7 (A6); no longer U4.3 (A2)
- net CELL_NET_STATUS: now also J5.13 (Pin_13), U4.14 (B6); no longer J5.25 (Pin_25), U4.18 (B2)
- net CELL_PWRKEY: now also J5.15 (Pin_15), U4.17 (B3); no longer J5.23 (Pin_23), U4.15 (B5)
- net CELL_PWRKEY_1V8: now also U3.15 (PWRKEY), U4.4 (A3); no longer U3.24 (ADC0), U4.6 (A5)
- net CELL_RESET_1V8: now also U3.17 (~{RESET}); no longer U3.2 (ADC1)
- net CELL_RX_1V8: now also U3.34 (MAIN_RXD), U4.3 (A2); no longer U3.96 (PON_TRIG), U4.7 (A6)
- net CELL_STATUS_1V8: now also U3.20 (STATUS), U4.6 (A5); no longer U3.75 (USB_BOOT), U4.4 (A3)
- net CELL_TX_1V8: now also U3.35 (MAIN_TXD), U4.1 (A1); no longer U4.8 (A7)
- net DBG_RX: now also J11.3 (Pin_3), J5.33 (Pin_33); no longer J11.1 (Pin_1), J5.5 (Pin_5)
- net USB_DP: now also J5.27 (Pin_27), U3.9 (USB_DP); no longer J5.11 (Pin_11)
- net 3V8_CELL: now reaches U2.5 (OUT)
- net 3V8_CELL: now also C13.1, C18.1, C19.1, U3.32 (VBAT_BB), U3.33 (VBAT_BB), U3.52 (VBAT_RF), U3.53 (VBAT_RF)
- net SHIFTER_OE: now reaches U4.10 (OE)
- net SHIFTER_OE: now also J5.29 (Pin_29), R6.1
- net VDD_EXT_1V8: now reaches U4.2 (VCCA)
- net VDD_EXT_1V8: now also C20.1, C23.1, U3.29 (VDD_EXT)
- net UART_RX_3V3: now reaches U4.20 (B1)
- net UART_RX_3V3: now also J5.10 (Pin_10)
- net +5V: now reaches J5.2 (Pin_2)
- net +5V: now also C10.1, C12.1, C14.1, C15.1, C16.1, C17.1, C6.2, C7.1, C8.1, C9.1, J4.8 (Pin_8), J5.4 (Pin_4), L2.1, L2.2, R2.1, U1.1 (VIN), U1.3 (EN), U2.1 (IN)
- net MPPT_BOOT: now reaches J2.11 (Pin_11)
- net MPPT_BOOT: now also C2.1
- net PV_IN: now reaches J2.15 (Pin_15)
- net PV_IN: now also C1.1, D1.1 (K), J2.14 (Pin_14)
- net USB_DM: now reaches U3.10 (USB_DM)
- net USB_DM: now also J5.28 (Pin_28)
- net ANT_IN: now reaches U3.60 (ANT_MAIN)
- net ANT_IN: now also C21.1, R5.1
- net VBAT: now reaches J4.5 (Pin_5)
- net VBAT: now also C3.1, C4.1, C5.1, J2.5 (Pin_5), J2.7 (Pin_7), J3.1 (Pin_1), J4.3 (Pin_3), R1.2
- net BUCK_FB: now reaches J4.7 (Pin_7)
- net BUCK_FB: now also R2.2, R3.1
- new net: J12.A4 (VBUS), J12.A9 (VBUS), J12.B4 (VBUS), J12.B9 (VBUS)
- new net ANT_MATCH: C22.1, J6.1 (In), R5.2
- new net BAT_SRP: J2.6 (Pin_6), L1.2, R1.1
- new net BUCK_BOOT: C6.1, J4.2 (Pin_2)
- new net BUCK_RT: J4.6 (Pin_6), R4.1
- new net CELL_EN: J5.11 (Pin_11), U2.3 (EN)
- new net CELL_RESET: J5.16 (Pin_16), U4.16 (B4)
- new net CELL_STATUS: J5.18 (Pin_18), U4.15 (B5)
- new net DBG_TX: J11.2 (Pin_2), J5.32 (Pin_32)
- new net GPIO25_VSYNC: J5.22 (Pin_22), J8.6 (Pin_6)
- new net MPPT_SW: C2.2, J2.10 (Pin_10), L1.1
- new net PV_RAW: D1.2 (A), J1.1 (Pin_1)
- new net SPI0_CE0: J5.24 (Pin_24), J8.2 (Pin_2)
- new net SPI0_MISO: J5.21 (Pin_21), J8.4 (Pin_4)
- new net SPI0_SCLK: J5.23 (Pin_23), J8.5 (Pin_5)
- new net UART_TX_3V3: J5.8 (Pin_8), U4.18 (B2)
- new net USB_CMSN_DM: J12.A7 (D-), J12.B7 (D-), J5.37 (Pin_37)
- new net USB_CMSN_DP: J12.A6 (D+), J12.B6 (D+), J5.36 (Pin_36)
- no-connect marks 42 -> 104

Commit message: 🐛 fix: per-component hash jitter to avoid ERC false-merge cascade
The y-mod-4 fix on power symbols handled cross-net y-coincidence between
power symbols, but the underlying grid-based component placement still gave
many components coincident pin y/x values, which KiCad's ERC then cascade-
merged into spurious cross-net "two power outputs" and "multiple net names"
errors.

Adding a per-component (dx, dy) jitter using prime moduli (17, 23) on the
component ref hash spreads pin positions enough to break the cascade. ERC
goes from 1 error + 2 warnings to 0 errors + 3 warnings. The remaining
warnings are pin_to_pin (Bidirectional ↔ Power output) and
multiple_net_names false-positives that don't affect the netlist.

Co-Authored-By: Claude Opus 4.7 (1M context) <noreply@anthropic.com>
Connections:
- net +3V3: now also J7.7 (I/O); no longer C29.1, J10.3 (Pin_3), J5.19 (Pin_19), J8.10 (Pin_10), J8.3 (Pin_3), U6.4 (AIN0)
- new net RAIN_AO: C29.1, J10.3 (Pin_3), U6.4 (AIN0)
- new net SPI0_MOSI: J5.19 (Pin_19), J8.3 (Pin_3)

Commit message: ✨ feat(anemometer): RS-485 wind sensor block + multi-sheet schematic
Adds IEEE 738 wind input via SP3485EN RS-485 transceiver. Sensor is a
field-replaceable SKU on the harness (Calypso ULP STD demo build, upgrade
to Vaisala WMT702 / Gill WO65 for low-wind sites). One PCB, two SKUs.

* theory.ipynb §6: derive dI/dV_w and dI/dphi from IEEE 738 sensitivity;
  required spec ±0.16 m/s, ±6°, ≤0.5 m/s threshold. Weibull climatology
  picks SKU per site.
* cad/netlist/anemometer.py: SP3485EN + 120Ω term + 680Ω bias + SM712
  TVS + 250 mA polyfuse + M12 5-pin connector, VBAT-fed.
* CM4: UART2 on GPIO0/1 (was USB2 placeholder), DE on GPIO6.
* cad/schematic/multi_sheet.py: hierarchical schematic generator —
  one .kicad_sch per block + root with sheet symbols. Per-sheet ERC
  scope bounds the y-coincidence false-merge bug (was 222 errors on
  single A1 sheet, now 0 functional + 2 cosmetic PWR_FLAG warnings).
* Root layout: A2 landscape, 3×2 grid, even spacing, PWR_FLAG bank
  centered above grid.

Co-Authored-By: Claude Opus 4.7 (1M context) <noreply@anthropic.com>
Parts:
- removed C1, C3: 22uF, Capacitor_SMD:C_1206_3216Metric, symbol Device:C
- removed C10, C11, C12, C13: 1uF, Capacitor_SMD:C_0402_1005Metric, symbol Device:C
- removed C14, C15, C16, C17, C19, C2, C20, C23, C24, C25, C26, C27, C28, C5, C6, C9: 100nF, Capacitor_SMD:C_0402_1005Metric, symbol Device:C
- removed C18: 4.7uF, Capacitor_SMD:C_0402_1005Metric, symbol Device:C
- removed C21, C22: DNP, Capacitor_SMD:C_0402_1005Metric, symbol Device:C
- removed C29: 10nF, Capacitor_SMD:C_0402_1005Metric, symbol Device:C
- removed C4: 4.7uF, Capacitor_SMD:C_0805_2012Metric, symbol Device:C
- removed C7: 470uF, Capacitor_SMD:CP_Elec_8x10, symbol Device:C_Polarized
- removed C8: 22uF, Capacitor_SMD:C_0805_2012Metric, symbol Device:C
- removed D1: SS34, Diode_SMD:D_SMA, symbol Device:D_Schottky
- removed J1: PV_IN, TerminalBlock_Phoenix:TerminalBlock_Phoenix_MKDS-1,5-2-5.08_1x02_P5.08mm_Horizontal, symbol Connector_Generic:Conn_01x02
- removed J10: YL-83, Connector_PinHeader_2.54mm:PinHeader_1x04_P2.54mm_Vertical, symbol Connector_Generic:Conn_01x04
- removed J11: DEBUG_UART, Connector_PinHeader_2.54mm:PinHeader_1x04_P2.54mm_Vertical, symbol Connector_Generic:Conn_01x04
- removed J12: USBC_COMMISSIONING, Connector_USB:USB_C_Receptacle_GCT_USB4085, symbol Connector:USB_C_Receptacle_USB2.0_14P
- removed J2: BQ24650, Package_DFN_QFN:HVQFN-16-1EP_3x3mm_P0.5mm_EP1.5x1.5mm, symbol Connector_Generic:Conn_02x08_Odd_Even
- removed J3: BAT, TerminalBlock_Phoenix:TerminalBlock_Phoenix_MKDS-1,5-2-5.08_1x02_P5.08mm_Horizontal, symbol Connector_Generic:Conn_01x02
- removed J4: LMR33630ADDA, Package_SO:HSOP-8-1EP_3.9x4.9mm_P1.27mm_EP2.41x3.1mm, symbol Connector_Generic:Conn_02x04_Odd_Even
- removed J5: CM4_J2, Connector_Hirose_DF40:Hirose_DF40HC(3.0)-40DS-0.4V_2x20_P0.4mm, symbol Connector_Generic:Conn_02x20_Odd_Even
- removed J6: U.FL, Connector_Coaxial:U.FL_Hirose_U.FL-R-SMT-1_Vertical, symbol Connector:Conn_Coaxial
- removed J7: SIM, Connector_Card:microSIM_JAE_SF53S006VCBR2000, symbol Connector:SIM_Card
- removed J8: FLIR_LEPTON_FFC, Connector_FFC-FPC:Hirose_FH12-14S-0.5SH_1x14-1MP_P0.50mm_Horizontal, symbol Connector_Generic:Conn_01x14
- removed J9: SI1145, Connector_PinHeader_2.54mm:PinHeader_1x05_P2.54mm_Vertical, symbol Connector_Generic:Conn_01x05
- removed L1: 6.8uH, Inductor_SMD:L_Bourns-SRN6028, symbol Device:L
- removed L2: 10uH, Inductor_SMD:L_Bourns-SRN8040_8x8.15mm, symbol Device:L
- removed R1: 20m, Resistor_SMD:R_1206_3216Metric, symbol Device:R
- removed R10, R11: 2.2k, Resistor_SMD:R_0402_1005Metric, symbol Device:R
- removed R12, R13: 5.1k, Resistor_SMD:R_0402_1005Metric, symbol Device:R
- removed R2: 39.2k, Resistor_SMD:R_0402_1005Metric, symbol Device:R
- removed R3, R7, R8, R9: 10k, Resistor_SMD:R_0402_1005Metric, symbol Device:R
- removed R4: 47k, Resistor_SMD:R_0402_1005Metric, symbol Device:R
- removed R5: 0R, Resistor_SMD:R_0402_1005Metric, symbol Device:R
- removed R6: 100k, Resistor_SMD:R_0402_1005Metric, symbol Device:R
- removed U1: AP2112K-3.3, Package_TO_SOT_SMD:SOT-23-5, symbol Regulator_Linear:AP2112K-3.3
- removed U2: LP5907MFX-3.8, Package_TO_SOT_SMD:SOT-23-5, symbol Regulator_Linear:LP5907MFX-3.3
- removed U3: BG770A-NA, RF_GSM:Quectel_BG95, symbol RF_GSM:BG95-M1
- removed U4: TXS0108E, Package_SO:TSSOP-20_4.4x6.5mm_P0.65mm, symbol Logic_LevelTranslator:TXS0108EPW
- removed U5: DHT22, Sensor:Aosong_DHT11_5.5x12.0_P2.54mm, symbol Sensor:DHT11
- removed U6: ADS1115, Package_SO:MSOP-10_3x3mm_P0.5mm, symbol Analog_ADC:ADS1115IDGS
Connections:
- no-connect marks 104 -> 0
Other:
- added sheet ANEMOMETER RS-485 (dlr_carrier-anemometer.kicad_sch)
- added sheet CELLULAR (dlr_carrier-cellular.kicad_sch)
- added sheet CM4 SoM (dlr_carrier-som.kicad_sch)
- added sheet CONNECTORS (dlr_carrier-connectors.kicad_sch)
- added sheet IEEE 738 SENSORS (dlr_carrier-sensors.kicad_sch)
- added sheet POWER (dlr_carrier-power.kicad_sch)
- note removed: "CELLULAR"
- note removed: "CM4 SoM"
- note removed: "CONNECTORS"
- note removed: "IEEE 738 SENSORS"
- note removed: "POWER"
